Commit message: Migrate kinematics functions into kinematics_manager.py

File: UsageTemplate/Resources/URDF/Demo_6/Demo_6.urdf (robot description, URDF)
Before this commit: robot Demo_6_Robot, 4 links, 3 joints
Joints:
- removed joint middle_proximal_2_rot_joint
- removed joint middle_proximal_rot_joint
- removed joint middle_to_top_joint
- added joint base_to_segment_1_joint: type revolute, parent base, child segment_1, origin xyz=0 0 0.0 rpy=0 0 0, axis 0 0 1, limit lower=0 upper=0 effort=0 velocity=0
- added joint middle_proximal_2_link_to_segment_3_joint: type revolute, parent middle_proximal_2_link, child segment_3, origin xyz=0 0 0.0 rpy=0 0 0, axis 0 0 1, limit lower=0 upper=0 effort=0 velocity=0
- added joint middle_proximal_link_to_segment_2_joint: type revolute, parent middle_proximal_link, child segment_2, origin xyz=0 0 0.0 rpy=0 0 0, axis 0 0 1, limit lower=0 upper=0 effort=0 velocity=0
- added joint segment_1_to_middle_proximal_link_joint: type revolute, parent segment_1, child middle_proximal_link, origin xyz=0 0 0.0 rpy=0 0 0, axis 0 0 1, limit lower=0 upper=0 effort=0 velocity=0
- added joint segment_2_to_middle_proximal_2_link_joint: type revolute, parent segment_2, child middle_proximal_2_link, origin xyz=0 0 0.0 rpy=0 0 0, axis 0 0 1, limit lower=0 upper=0 effort=0 velocity=0
- added joint segment_3_to_top_link_joint: type revolute, parent segment_3, child top_link, origin xyz=0 0 0.0 rpy=0 0 0, axis 0 0 1, limit lower=0 upper=0 effort=0 velocity=0

Commit message: Add scale element

File: UsageTemplate/Resources/URDF/Demo_6/Demo_6.urdf (robot description, URDF)
Before this commit: robot Demo_6_Robot, 4 links, 6 joints
Joints:
- joint base_to_segment_1_joint: limit lower=0 upper=0 effort=0 velocity=0 -> (none)
- joint middle_proximal_2_link_to_segment_3_joint: limit lower=0 upper=0 effort=0 velocity=0 -> (none)
- joint middle_proximal_link_to_segment_2_joint: limit lower=0 upper=0 effort=0 velocity=0 -> (none)
- joint segment_1_to_middle_proximal_link_joint: limit lower=0 upper=0 effort=0 velocity=0 -> (none)
- joint segment_2_to_middle_proximal_2_link_joint: limit lower=0 upper=0 effort=0 velocity=0 -> (none)
- joint segment_3_to_top_link_joint: limit lower=0 upper=0 effort=0 velocity=0 -> (none)
